File: office_amp/Power.kicad_sch (KiCad schematic)
At the start: 37 parts, among them J1 Jack-DC, Q1 DMT6012LSS, U1 LM74700, U2 LM7805_TO220, U4 TBA_2-2421, U7 LM7812_TO220

Commit message: changes from tim and josef, prototype
Parts:
- removed C37, C7: 100nF, Capacitor_SMD:C_0805_2012Metric_Pad1.18x1.45mm_HandSolder, symbol Device:C
- removed C43: 2µ2F, Capacitor_SMD:C_0805_2012Metric_Pad1.18x1.45mm_HandSolder, symbol Device:C
- removed R32, R33: 10k, Resistor_SMD:R_0805_2012Metric_Pad1.20x1.40mm_HandSolder, symbol Device:R
- added C37, C7: 10µF, Capacitor_THT:CP_Radial_D5.0mm_P2.00mm, symbol Device:C_Polarized
- added C43: 470µF, Capacitor_THT:CP_Radial_D10.0mm_P5.00mm, symbol Device:CP
- added C46: 100µF, Capacitor_THT:CP_Radial_D13.0mm_P5.00mm, symbol Device:CP
- added C47, C48: 1000µF, Capacitor_THT:CP_Radial_D13.0mm_P5.00mm, symbol Device:CP
- added D4: 18TQ045, Package_TO_SOT_THT:TO-220-2_Vertical, symbol Device:D_Schottky
- added J4: Conn_01x08_Pin, symbol Connector:Conn_01x08_Pin
- added L4, L8: 56µH, Inductor_THT:L_Axial_L16.0mm_D6.3mm_P25.40mm_Horizontal_Fastron_VHBCC, symbol Device:L
- added L7: 12µH, office_amp:L_Radial_D10.0mm_P5.00mm, symbol Device:L
- added R40: 1k, Resistor_SMD:R_0805_2012Metric_Pad1.20x1.40mm_HandSolder, symbol Device:R
- added R41: 3k2, Resistor_SMD:R_0805_2012Metric_Pad1.20x1.40mm_HandSolder, symbol Device:R
- added TP6: TestPoint, TestPoint:TestPoint_Pad_D1.0mm, symbol Connector:TestPoint
- added U13: LM2576HVT-ADJ, Package_TO_SOT_THT:TO-220-5_Vertical, symbol Regulator_Switching:LM2576HVT-ADJ
- U7: value LM7812_TO220 -> VXO78012_TO220
Connections:
- net +12V: now also C7.1, J4.3 (Pin_3)
- net +5V: now also J4.4 (Pin_4)
- net +5VA: now also J4.6 (Pin_6)
- net -5VA: now also J4.7 (Pin_7)
- net GNDREF: now also C37.2, C43.2, C46.2, C47.2, C48.2, C7.2, J4.1 (Pin_1), L4.2, R41.1
- net GND_Input: now also J4.8 (Pin_8)
- net V+: now also C46.1, J4.2 (Pin_2), L8.1, U13.1 (VIN); no longer C5.1, U7.1 (VI)
- new net: C43.1, C5.1, L7.1, L8.2
- new net: C37.1, L7.2, U7.1 (VI)
- new net: D4.1 (K), L4.1, U13.2 (OUT)
- new net: R40.1, R41.2, U13.4 (FB)
- new net -5V: C47.1, C48.1, D4.2 (A), J4.5 (Pin_5), R40.2, TP6.1, U13.3 (GND), U13.5 (~{ON}/OFF)
Other:
- note added: "-5 V DCDC"
- moved on the sheet: C5, TP7, U7
