File: office_amp/_autosave-office_amp.kicad_pcb (KiCad board)
At the start: 2 copper layers, 160 x 100 mm, 161 parts, among them J1 Jack-DC, J2 Conn_01x03_Female, J3 Conn_02x07_Odd_Even, J7 Screw_Terminal_01x04, J8 Conn_01x03_Female, K1 V23079-A1003-B301, K2 V23079-A1003-B301, K3 V23079-A1003-B301, K4 V23079-A1003-B301, Q1 DMT6012LSS, Q10 BSS138, Q11 BSS138, Q2 BC858, Q3 BC858, Q4 BC850, Q5 BC850, Q6 BC856, Q7 BC850, Q8 BC856, Q9 BC856, U1 LM74700, U10 DS1882E, U11 TL082, U12 TL082, U13 LM2576HVT-ADJ, U2 LM7805_TO220, U3 TL082, U4 TBA_2-2421, U5 MH-M18, U6 TPA3123D2, U7 VXO78012_TO220, U8 IL300, U9 IL300

Commit message: changes from tim and josef, prototype
Parts:
- C6, C8: moved to B.Cu
- moved TP10 28.6 mm to (202.0, 94.5)
- moved TP7 20.1 mm to (224.5, 100.0), turned to 0 degrees
- moved C8 12.2 mm to (222.0, 103.1), turned to 180 degrees
- moved TP11 11.8 mm to (196.0, 94.0)
- moved TP6 6.68 mm to (169.5, 82.0)
- moved TP13 5.40 mm to (187.5, 93.0), turned to 0 degrees
- moved C6 4.45 mm to (217.5, 93.1), turned to 0 degrees
- moved U2 2.09 mm to (218.0, 98.5), turned to 0 degrees
- moved C7 1.80 mm to (217.5, 86.0)
Routing:
- net +5V: track 0.00 -> 105.0 mm, vias 0 -> 1
- net GNDREF: track 224.0 -> 275.2 mm
- net Net-(C43-Pad1): track 0.00 -> 31.8 mm
- net +12V: track 0.00 -> 15.6 mm
- net Net-(U7-VI): track 0.00 -> 14.6 mm
